File: High_Amp_PCB_Designs/KiCAD_Design/High_AMP_BLDC_Control/High_AMP_BLDC_Control.kicad_pcb (KiCad board)
At the start: 2 copper layers, 42 x 29 mm, 4 parts

Commit message: :construction: Python script ongoing.
Parts:
- removed R1, R2, R3, R4: R, Resistor_SMD:R_0201_0603Metric_Pad0.64x0.40mm_HandSolder
- added Q1: NMOS, FOOTPRINT:MOSFET_CSD19531Q5A, F.Cu at (84.2, 85.6)
Routing:
- net Net-(R2-Pad2): track 15.2 -> 0.00 mm
- net Net-(R1-Pad2): track 12.8 -> 0.00 mm
